Commit message: noetic changes

File: configs/gazebo_files/urdf/component_snippets.xacro (robot description, xacro)
@@ -37,5 +37,5 @@
       <inertial>
          <mass value="0.01" />
-         <inertia ixx="1e-6" ixy="0.0" ixz="0.0" iyy="1e-6" iyz="0.0" izz="1e-6" />
+         <inertia ixx="0.0" ixy="0.0" ixz="0.0" iyy="0.0" iyz="0.0" izz="0.0" />
       </inertial>
       <visual name="visual">
@@ -51,9 +51,9 @@
     </joint>
     <gazebo reference="${namespace}/hokuyo_link">
-    <sensor type="gpu_ray" name="head_hokuyo_sensor">
+    <sensor type="ray" name="head_hokuyo_sensor">
       <pose>0 0 0 0 0 0</pose>
       <visualize>false</visualize>
       <update_rate>40</update_rate>
-      <gpu_ray>
+      <ray>
         <scan>
           <horizontal>
@@ -78,5 +78,5 @@
           <stddev>0.01</stddev>
         </noise>
-      </gpu_ray>
+      </ray>
       <plugin name="gazebo_ros_head_hokuyo_controller" filename="libgazebo_ros_laser.so">
         <topicName>/drone111/scan</topicName>

File: configs/gazebo_files/urdf/hummingbird_laser_base.xacro (robot description, xacro)
@@ -44,5 +44,5 @@
   </gazebo>
   <xacro:camera_macro
-   namespace="drone111"
+   namespace="${namespace}"
    parent_link="${namespace}/base_link"
    camera_suffix="front"
